Commit message: added ros2_controllers

File: gazebo_rby/urdf/robots/rby_gazebo.urdf.xacro (robot description, xacro)
@@ -7,193 +7,313 @@
     <!-- Add Gazebo-specific sensor tags -->
     <xacro:lidar_gazebo frame="lidar_link" topic_name="scan" sensor_name="lidar_sensor" />
-    <!-- Macro para aplicar propiedades a todos los joints -->
-    <xacro:macro name="add_joint_properties">
-        <xacro:gazebo_joint_properties joint="torso_0" />
-        <xacro:gazebo_joint_properties joint="torso_1" />
-        <xacro:gazebo_joint_properties joint="torso_2" />
-        <xacro:gazebo_joint_properties joint="torso_3" />
-        <xacro:gazebo_joint_properties joint="torso_4" />
-        <xacro:gazebo_joint_properties joint="torso_5" />
-        <xacro:gazebo_joint_properties joint="left_wheel" />
-        <xacro:gazebo_joint_properties joint="right_wheel" />
-        <xacro:gazebo_joint_properties joint="right_arm_0" />
-        <xacro:gazebo_joint_properties joint="right_arm_1" />
-        <xacro:gazebo_joint_properties joint="right_arm_2" />
-        <xacro:gazebo_joint_properties joint="right_arm_3" />
-        <xacro:gazebo_joint_properties joint="right_arm_4" />
-        <xacro:gazebo_joint_properties joint="right_arm_5" />
-        <xacro:gazebo_joint_properties joint="right_arm_6" />
-        <xacro:gazebo_joint_properties joint="left_arm_0" />
-        <xacro:gazebo_joint_properties joint="left_arm_1" />
-        <xacro:gazebo_joint_properties joint="left_arm_2" />
-        <xacro:gazebo_joint_properties joint="left_arm_3" />
-        <xacro:gazebo_joint_properties joint="left_arm_4" />
-        <xacro:gazebo_joint_properties joint="left_arm_5" />
-        <xacro:gazebo_joint_properties joint="left_arm_6" />
-        <xacro:gazebo_joint_properties joint="tool_right" />
-        <xacro:gazebo_joint_properties joint="FT_Sensor_END_right" />
-        <xacro:gazebo_joint_properties joint="gripper_finger_r1" />
-        <xacro:gazebo_joint_properties joint="gripper_finger_r2" />
-        <xacro:gazebo_joint_properties joint="tool_left" />
-        <xacro:gazebo_joint_properties joint="FT_Sensor_END_left" />
-        <xacro:gazebo_joint_properties joint="gripper_finger_l1" />
-        <xacro:gazebo_joint_properties joint="gripper_finger_l2" />
-        <xacro:gazebo_joint_properties joint="head_base" />
-        <xacro:gazebo_joint_properties joint="head_0" />
-        <xacro:gazebo_joint_properties joint="head_1" />
-        <xacro:gazebo_joint_properties joint="lidar" />
-    </xacro:macro>
-    <xacro:macro name="gazebo_joint_properties" params="joint">
-        <gazebo reference="${joint}">
-            <stopCfm>0.1</stopCfm>
-            <stopErp>0.8</stopErp>
-            <implicitSpringDamper>true</implicitSpringDamper>
-            <damping>0.7</damping>
-            <friction>0.5</friction>
-        </gazebo>
-    </xacro:macro>
-    <!-- Llamar el macro -->
-    <xacro:add_joint_properties />
-    <!-- Plugin de GAZEBO HARMONIC -->
-    <!-- Plugin de GAZEBO HARMONIC -->
-    <!-- Plugin de GAZEBO HARMONIC -->
+    <ros2_control name="GazeboSimSystem" type="system">
+        <hardware>
+            <plugin>gz_ros2_control/GazeboSimSystem</plugin>
+        </hardware>
+        <joint name="right_wheel">
+            <command_interface name="position" />
+            <state_interface name="position">
+                <param name="initial_value">0.0</param>
+            </state_interface>
+            <state_interface name="velocity" />
+            <state_interface name="effort" />
+        </joint>
+        <joint name="left_wheel">
+            <command_interface name="position" />
+            <state_interface name="position">
+                <param name="initial_value">0.0</param>
+            </state_interface>
+            <state_interface name="velocity" />
+            <state_interface name="effort" />
+        </joint>
+        <joint name="torso_0">
+            <command_interface name="position">
+                <param name="min">-0.261799388</param>
+                <param name="max">0.261799388</param>
+            </command_interface>
+            <state_interface name="position">
+                <param name="initial_value">0.0</param>
+            </state_interface>
+            <state_interface name="velocity" />
+            <state_interface name="effort" />
+        </joint>
+        <joint name="torso_1">
+            <command_interface name="position">
+                <param name="min">-0.523598776</param>
+                <param name="max">1.570796327</param>
+            </command_interface>
+            <state_interface name="position">
+                <param name="initial_value">0.0</param>
+            </state_interface>
+            <state_interface name="velocity" />
+            <state_interface name="effort" />
+        </joint>
+        <joint name="torso_2">
+            <command_interface name="position">
+                <param name="min">-2.617993878</param>
+                <param name="max">1.570796327</param>
+            </command_interface>
+            <state_interface name="position">
+                <param name="initial_value">0.0</param>
+            </state_interface>
+            <state_interface name="velocity" />
+            <state_interface name="effort" />
+        </joint>
+        <joint name="torso_3">
+            <command_interface name="position">
+                <param name="min">-0.785398163</param>
+                <param name="max">1.570796327</param>
+            </command_interface>
+            <state_interface name="position">
+                <param name="initial_value">0.0</param>
+            </state_interface>
+            <state_interface name="velocity" />
+            <state_interface name="effort" />
+        </joint>
+        <joint name="torso_4">
+            <command_interface name="position">
+                <param name="min">-0.523598776</param>
+                <param name="max">0.523598776</param>
+            </command_interface>
+            <state_interface name="position">
+                <param name="initial_value">0.0</param>
+            </state_interface>
+            <state_interface name="velocity" />
+            <state_interface name="effort" />
+        </joint>
+        <joint name="torso_5">
+            <command_interface name="position">
+                <param name="min">-2.35619449</param>
+                <param name="max">2.35619449</param>
+            </command_interface>
+            <state_interface name="position">
+                <param name="initial_value">0.0</param>
+            </state_interface>
+            <state_interface name="velocity" />
+            <state_interface name="effort" />
+        </joint>
+        <joint name="right_arm_0">
+            <command_interface name="position">
+                <param name="min">-3.141592654</param>
+                <param name="max">3.141592654</param>
+            </command_interface>
+            <state_interface name="position">
+                <param name="initial_value">0.0</param>
+            </state_interface>
+            <state_interface name="velocity" />
+            <state_interface name="effort" />
+        </joint>
+        <joint name="right_arm_1">
+            <command_interface name="position">
+                <param name="min">-3.141592654</param>
+                <param name="max">0.017453293</param>
+            </command_interface>
+            <state_interface name="position">
+                <param name="initial_value">0.0</param>
+            </state_interface>
+            <state_interface name="velocity" />
+            <state_interface name="effort" />
+        </joint>
+        <joint name="right_arm_2">
+            <command_interface name="position">
+                <param name="min">-3.141592654</param>
+                <param name="max">3.141592654</param>
+            </command_interface>
+            <state_interface name="position">
+                <param name="initial_value">0.0</param>
+            </state_interface>
+            <state_interface name="velocity" />
+            <state_interface name="effort" />
+        </joint>
+        <joint name="right_arm_3">
+            <command_interface name="position">
+                <param name="min">-2.617993878</param>
+                <param name="max">0.017453293</param>
+            </command_interface>
+            <state_interface name="position">
+                <param name="initial_value">0.0</param>
+            </state_interface>
+            <state_interface name="velocity" />
+            <state_interface name="effort" />
+        </joint>
+        <joint name="right_arm_4">
+            <command_interface name="position">
+                <param name="min">-3.141592654</param>
+                <param name="max">3.141592654</param>
+            </command_interface>
+            <state_interface name="position">
+                <param name="initial_value">0.0</param>
+            </state_interface>
+            <state_interface name="velocity" />
+            <state_interface name="effort" />
+        </joint>
+        <joint name="right_arm_5">
+            <command_interface name="position">
+                <param name="min">-1.570796327</param>
+                <param name="max">1.919862177</param>
+            </command_interface>
+            <state_interface name="position">
+                <param name="initial_value">0.0</param>
+            </state_interface>
+            <state_interface name="velocity" />
+            <state_interface name="effort" />
+        </joint>
+        <joint name="right_arm_6">
+            <command_interface name="position">
+                <param name="min">-2.705260340</param>
+                <param name="max">2.705260340</param>
+            </command_interface>
+            <state_interface name="position">
+                <param name="initial_value">0.0</param>
+            </state_interface>
+            <state_interface name="velocity" />
+            <state_interface name="effort" />
+        </joint>
+        <joint name="left_arm_0">
+            <command_interface name="position">
+                <param name="min">-3.141592654</param>
+                <param name="max">3.141592654</param>
+            </command_interface>
+            <state_interface name="position">
+                <param name="initial_value">0.0</param>
+            </state_interface>
+            <state_interface name="velocity" />
+            <state_interface name="effort" />
+        </joint>
+        <joint name="left_arm_1">
+            <command_interface name="position">
+                <param name="min">-0.017453293</param>
+                <param name="max">3.141592654</param>
+            </command_interface>
+            <state_interface name="position">
+                <param name="initial_value">0.0</param>
+            </state_interface>
+            <state_interface name="velocity" />
+            <state_interface name="effort" />
+        </joint>
+        <joint name="left_arm_2">
+            <command_interface name="position">
+                <param name="min">-3.141592654</param>
+                <param name="max">3.141592654</param>
+            </command_interface>
+            <state_interface name="position">
+                <param name="initial_value">0.0</param>
+            </state_interface>
+            <state_interface name="velocity" />
+            <state_interface name="effort" />
+        </joint>
+        <joint name="left_arm_3">
+            <command_interface name="position">
+                <param name="min">-2.617993878</param>
+                <param name="max">0.017453293</param>
+            </command_interface>
+            <state_interface name="position">
+                <param name="initial_value">0.0</param>
+            </state_interface>
+            <state_interface name="velocity" />
+            <state_interface name="effort" />
+        </joint>
+        <joint name="left_arm_4">
+            <command_interface name="position">
+                <param name="min">-3.141592654</param>
+                <param name="max">3.141592654</param>
+            </command_interface>
+            <state_interface name="position">
+                <param name="initial_value">0.0</param>
+            </state_interface>
+            <state_interface name="velocity" />
+            <state_interface name="effort" />
+        </joint>
+        <joint name="left_arm_5">
+            <command_interface name="position">
+                <param name="min">-1.570796327</param>
+                <param name="max">1.919862177</param>
+            </command_interface>
+            <state_interface name="position">
+                <param name="initial_value">0.0</param>
+            </state_interface>
+            <state_interface name="velocity" />
+            <state_interface name="effort" />
+        </joint>
+        <joint name="left_arm_6">
+            <command_interface name="position">
+                <param name="min">-2.705260340</param>
+                <param name="max">2.705260340</param>
+            </command_interface>
+            <state_interface name="position">
+                <param name="initial_value">0.0</param>
+            </state_interface>
+            <state_interface name="velocity" />
+            <state_interface name="effort" />
+        </joint>
+        <joint name="gripper_finger_r1">
+            <command_interface name="position">
+                <param name="min">-0.05</param>
+                <param name="max">0.0</param>
+            </command_interface>
+            <state_interface name="position">
+                <param name="initial_value">0.0</param>
+            </state_interface>
+            <state_interface name="velocity" />
+            <state_interface name="effort" />
+        </joint>
+        <joint name="gripper_finger_r2">
+            <command_interface name="position">
+                <param name="min">0.0</param>
+                <param name="max">0.05</param>
+            </command_interface>
+            <state_interface name="position">
+                <param name="initial_value">0.0</param>
+            </state_interface>
+            <state_interface name="velocity" />
+            <state_interface name="effort" />
+        </joint>
+        <joint name="gripper_finger_l1">
+            <command_interface name="position">
+                <param name="min">-0.05</param>
+                <param name="max">0.0</param>
+            </command_interface>
+            <state_interface name="position">
+                <param name="initial_value">0.0</param>
+            </state_interface>
+            <state_interface name="velocity" />
+            <state_interface name="effort" />
+        </joint>
+        <joint name="gripper_finger_l2">
+            <command_interface name="position">
+                <param name="min">0.0</param>
+                <param name="max">0.05</param>
+            </command_interface>
+            <state_interface name="position">
+                <param name="initial_value">0.0</param>
+            </state_interface>
+            <state_interface name="velocity" />
+            <state_interface name="effort" />
+        </joint>
+        <joint name="head_0">
+            <command_interface name="position">
+            <param name="min">-2.08567</param>
+            <param name="max">2.08567</param>
+            </command_interface>
+            <state_interface name="position">
+            <param name="initial_value">0.0</param>
+            </state_interface>
+            <state_interface name="velocity"/>
+        </joint>
+        <joint name="head_1">
+            <command_interface name="position">
+            <param name="min">-2.08567</param>
+            <param name="max">2.08567</param>
+            </command_interface>
+            <state_interface name="position">
+            <param name="initial_value">0.0</param>
+            </state_interface>
+            <state_interface name="velocity"/>
+        </joint>
+    </ros2_control>
     <gazebo>
-        <plugin
-            name="gz_ros2_control::GazeboSimROS2ControlPlugin"
-            filename="libgz_ros2_control-system.so">
-            <ros2_control>
-                <param name="robot_description">robot_description</param>
-            </ros2_control>
+        <plugin filename="gz_ros2_control-system" name="gz_ros2_control::GazeboSimROS2ControlPlugin">
+            <parameters>$(find gazebo_rby)/config/rby_controller_manager.yaml</parameters>
         </plugin>
     </gazebo>
-    <!-- ros2_control hardware - using mock system -->
-    <ros2_control name="rby_system" type="system">
-        <hardware>
-            <plugin>mock_components/GenericSystem</plugin>
-        </hardware>
-        <!-- WHEELS -->
-        <joint name="left_wheel">
-            <command_interface name="velocity" />
-            <state_interface name="velocity" />
-            <state_interface name="position" />
-        </joint>
-        <joint name="right_wheel">
-            <command_interface name="velocity" />
-            <state_interface name="velocity" />
-            <state_interface name="position" />
-        </joint>
-        <!-- TORSO JOINTS -->
-        <joint name="torso_0">
-            <command_interface name="position" />
-            <state_interface name="position" />
-            <state_interface name="velocity" />
-        </joint>
-        <joint name="torso_1">
-            <command_interface name="position" />
-            <state_interface name="position" />
-            <state_interface name="velocity" />
-        </joint>
-        <joint name="torso_2">
-            <command_interface name="position" />
-            <state_interface name="position" />
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
Commit message: added ros2_controllers

File: gazebo_rby/urdf/robots/rby_gazebo.urdf.xacro (robot description, xacro)
@@ -11,20 +11,4 @@
             <plugin>gz_ros2_control/GazeboSimSystem</plugin>
         </hardware>
-        <joint name="right_wheel">
-            <command_interface name="position" />
-            <state_interface name="position">
-                <param name="initial_value">0.0</param>
-            </state_interface>
-            <state_interface name="velocity" />
-            <state_interface name="effort" />
-        </joint>
-        <joint name="left_wheel">
-            <command_interface name="position" />
-            <state_interface name="position">
-                <param name="initial_value">0.0</param>
-            </state_interface>
-            <state_interface name="velocity" />
-            <state_interface name="effort" />
-        </joint>
         <joint name="torso_0">
             <command_interface name="position">
@@ -317,3 +301,28 @@
         </plugin>
     </gazebo>
+    <gazebo>
+        <plugin
+        filename="gz-sim-diff-drive-system"
+        name="gz::sim::systems::DiffDrive">
+        <left_joint>left_wheel</left_joint>
+        <right_joint>right_wheel</right_joint>
+        <wheel_separation>0.48</wheel_separation>
+        <wheel_radius>0.1</wheel_radius>
+        <topic>cmd_vel</topic>
+        <odom_topic>odom</odom_topic>
+        <frame_id>odom</frame_id>
+        <child_frame_id>base_link</child_frame_id>
+        <odom_publish_frequency>30</odom_publish_frequency>
+        <tf_topic>/tf</tf_topic>
+        </plugin>
+    </gazebo>
+    <gazebo>
+        <plugin
+        filename="gz-sim-joint-state-publisher-system"
+        name="gz::sim::systems::JointStatePublisher">
+        <topic>joint_states</topic>
+        <joint_name>left_wheel</joint_name>
+        <joint_name>right_wheel</joint_name>
+        </plugin>
+    </gazebo>
 </robot>

File: urdf_rby/urdf/robots/rby.urdf.xacro (robot description, xacro)
@@ -6,7 +6,4 @@
         <xacro:property name="wheel_radius" value="0.1" />
         <xacro:include filename="$(find urdf_rby)/urdf/sensors/lidar.urdf.xacro" />
-        <!-- Mobile base properties -->
-        <mobile type="differential" xyz="0.228 0 0" rpy="0 0 0" joints="right_wheel left_wheel"
-            params="0.53 0.1" />
         <!-- Base Link -->
         <link name="base">
@@ -25,5 +22,5 @@
                 <origin rpy="0 0 0" xyz="0 0 0.1" />
                 <geometry>
-                    <box size="0.5 0.4 0.2" />
+                    <box size="0.5 0.4 0.17" />
                 </geometry>
             </collision>
@@ -32,5 +29,5 @@
         <link name="wheel_r">
             <inertial>
-                <mass value="1.37783736" />
+                <mass value="10.37783736" />
                 <origin rpy="0 0 0" xyz="0.0 -0.00073938 0.0" />
                 <inertia ixx="0.00426657" ixy="0.0" ixz="0.0"
@@ -42,9 +39,14 @@
                 </geometry>
             </visual>
+            <collision>
+                <geometry>
+                    <mesh filename="package://urdf_rby/meshes/WHEEL.dae" />
+                </geometry>
+            </collision>
         </link>
         <!-- Left Wheel Link -->
         <link name="wheel_l">
             <inertial>
-                <mass value="1.37783736" />
+                <mass value="10.37783736" />
                 <origin rpy="0 0 0" xyz="0.0 0.00073938 0.0" />
                 <inertia ixx="0.00426657" ixy="0.0" ixz="0.0"
@@ -56,4 +58,9 @@
                 </geometry>
             </visual>
+            <collision>
+                <geometry>
+                    <mesh filename="package://urdf_rby/meshes/WHEEL.dae" />
+                </geometry>
+            </collision>
         </link>
         <!-- Torso Links -->
@@ -592,5 +599,5 @@
             <origin rpy="0.0 0.0 0.0" xyz="0.228 -0.265 0.1" />
             <axis xyz="0 -1 0" />
-            <limit effort="100.0" velocity="15.707963268" />
+            <limit effort="1000.0" velocity="500.707963268" />
         </joint>
         <joint name="left_wheel" type="continuous">
@@ -599,5 +606,5 @@
             <origin rpy="0.0 0.0 0.0" xyz="0.228 0.265 0.1" />
             <axis xyz="0 -1 0" />
-            <limit effort="100.0" velocity="15.707963268" />
+            <limit effort="1000.0" velocity="500.707963268" />
         </joint>
         <!-- Torso Joints -->
