Commit message: fix ruedas locas

File: gazebo_rby/urdf/robots/rby_gazebo.urdf.xacro (robot description, xacro)
@@ -324,4 +324,8 @@
         <joint_name>left_wheel</joint_name>
         <joint_name>right_wheel</joint_name>
+        <joint_name>left_rear_wheel1</joint_name>
+        <joint_name>left_rear_wheel2</joint_name>
+        <joint_name>right_rear_wheel1</joint_name>
+        <joint_name>right_rear_wheel2</joint_name>
         </plugin>
     </gazebo>

File: urdf_rby/urdf/robots/rby.urdf.xacro (robot description, xacro)
@@ -2,5 +2,4 @@
 <robot xmlns:xacro="http://www.ros.org/wiki/xacro" name="rby_A_v1.0">
     <xacro:macro name="rby" params="name use_sensors:=true">
-        <!-- Properties for easy parameter management -->
         <xacro:property name="wheel_base" value="0.53" />
         <xacro:property name="wheel_radius" value="0.1" />
@@ -16,5 +15,5 @@
             <visual>
                 <geometry>
-                    <mesh filename="package://urdf_rby/meshes/base.dae" />
+                    <mesh filename="package://urdf_rby/meshes/untitled.dae" />
                 </geometry>
             </visual>
@@ -62,4 +61,80 @@
                     <mesh filename="package://urdf_rby/meshes/WHEEL.dae" />
                 </geometry>
+            </collision>
+        </link>
+        <link name="wheel_rear_r1">
+            <inertial>
+                <mass value="3.0" />
+                <origin rpy="0 0 0" xyz="0.0 -0.00073938 0.0" />
+                <inertia ixx="0.001" ixy="0.0" ixz="0.0"
+                    iyy="0.002" iyz="0.0" izz="0.001" />
+            </inertial>
+            <visual>
+                <geometry>
+                    <mesh filename="package://urdf_rby/meshes/WHEEL.dae" scale=".35 .35 .35" />
+                </geometry>
+            </visual>
+            <collision>
+                <geometry>
+                    <cylinder radius="0.04" length="0.03" />
+                </geometry>
+                <origin rpy="1.5708 0 0" xyz="0 0 0" />
+            </collision>
+        </link>
+        <link name="wheel_rear_r2">
+            <inertial>
+                <mass value="3.0" />
+                <origin rpy="0 0 0" xyz="0.0 -0.00073938 0.0" />
+                <inertia ixx="0.001" ixy="0.0" ixz="0.0"
+                    iyy="0.002" iyz="0.0" izz="0.001" />
+            </inertial>
+            <visual>
+                <geometry>
+                    <mesh filename="package://urdf_rby/meshes/WHEEL.dae" scale=".35 .35 .35" />
+                </geometry>
+            </visual>
+            <collision>
+                <geometry>
+                    <cylinder radius="0.04" length="0.03" />
+                </geometry>
+                <origin rpy="1.5708 0 0" xyz="0 0 0" />
+            </collision>
+        </link>
+        <link name="wheel_rear_l1">
+            <inertial>
+                <mass value="3.0" />
+                <origin rpy="0 0 0" xyz="0.0 0.00073938 0.0" />
+                <inertia ixx="0.001" ixy="0.0" ixz="0.0"
+                    iyy="0.002" iyz="0.0" izz="0.001" />
+            </inertial>
+            <visual>
+                <geometry>
+                    <mesh filename="package://urdf_rby/meshes/WHEEL.dae" scale=".33 .33 .33" />
+                </geometry>
+            </visual>
+            <collision>
+                <geometry>
+                    <cylinder radius="0.04" length="0.03" />
+                </geometry>
+                <origin rpy="1.5708 0 0" xyz="0 0 0" />
+            </collision>
+        </link>
+        <link name="wheel_rear_l2">
+            <inertial>
+                <mass value="3.0" />
+                <origin rpy="0 0 0" xyz="0.0 0.00073938 0.0" />
+                <inertia ixx="0.001" ixy="0.0" ixz="0.0"
+                    iyy="0.002" iyz="0.0" izz="0.001" />
+            </inertial>
+            <visual>
+                <geometry>
+                    <mesh filename="package://urdf_rby/meshes/WHEEL.dae" scale=".33 .33 .33" />
+                </geometry>
+            </visual>
+            <collision>
+                <geometry>
+                    <cylinder radius="0.04" length="0.03" />
+                </geometry>
+                <origin rpy="1.5708 0 0" xyz="0 0 0" />
             </collision>
         </link>
@@ -598,5 +673,5 @@
             <child link="wheel_r" />
             <origin rpy="0.0 0.0 0.0" xyz="0.228 -0.265 0.1" />
-            <axis xyz="0 -1 0" />
+            <axis xyz="0 1 0" />
             <limit effort="1000.0" velocity="500.707963268" />
         </joint>
@@ -605,6 +680,34 @@
             <child link="wheel_l" />
             <origin rpy="0.0 0.0 0.0" xyz="0.228 0.265 0.1" />
-            <axis xyz="0 -1 0" />
+            <axis xyz="0 1 0" />
             <limit effort="1000.0" velocity="500.707963268" />
+        </joint>
+        <joint name="right_rear_wheel1" type="continuous">
+            <parent link="base" />
+            <child link="wheel_rear_r1" />
+            <origin rpy="0.0 0.0 0.0" xyz="-0.277 -0.09999999 0.05" />
+            <axis xyz="0 1 0" />
+            <limit effort="100.0" velocity="500.707963268" />
+        </joint>
+        <joint name="right_rear_wheel2" type="continuous">
+            <parent link="base" />
+            <child link="wheel_rear_r2" />
+            <origin rpy="0.0 0.0 0.0" xyz="-0.277 -0.07 0.05" />
+            <axis xyz="0 1 0" />
+            <limit effort="100.0" velocity="500.707963268" />
+        </joint>
+        <joint name="left_rear_wheel1" type="continuous">
+            <parent link="base" />
+            <child link="wheel_rear_l1" />
+            <origin rpy="0.0 0.0 0.0" xyz="-0.277 0.09999999 0.05" />
+            <axis xyz="0 1 0" />
+            <limit effort="100.0" velocity="500.707963268" />
+        </joint>
+        <joint name="left_rear_wheel2" type="continuous">
+            <parent link="base" />
+            <child link="wheel_rear_l2" />
+            <origin rpy="0.0 0.0 0.0" xyz="-0.277 0.07 0.05" />
+            <axis xyz="0 1 0" />
+            <limit effort="100.0" velocity="500.707963268" />
         </joint>
         <!-- Torso Joints -->
