Commit message: [Fix]: structure and launch fixed

File: urdf_rby/urdf/robots/rby.urdf.xacro (robot description, xacro)
@@ -6,4 +6,11 @@
         <xacro:property name="wheel_radius" value="0.1" />
         <xacro:include filename="$(find urdf_rby)/urdf/sensors/lidar.urdf.xacro" />
+        <!-- Nuevo root sin inercia -->
+        <link name="base_footprint"/>
+        <joint name="base_footprint_to_base" type="fixed">
+            <parent link="base_footprint"/>
+            <child link="base"/>
+            <origin xyz="0 0 0" rpy="0 0 0"/>
+        </joint>
         <!-- Base Link -->
         <link name="base">
@@ -621,5 +628,5 @@
             <origin rpy="0.0 0.0 0.0" xyz="0.0 0.0 0.0" />
             <axis xyz="0 1 0" />
-            <limit effort="270.0" velocity="2.09439510" lower="-0.523598776" upper="1.570796327" />
+            <limit effort="270.0" velocity="2.09439510" lower="-0.523598776" upper="0.523598776" />
         </joint>
         <joint name="torso_2" type="revolute">
@@ -628,5 +635,5 @@
             <origin rpy="0.0 0.0 0.0" xyz="0.0 0.0 0.350" />
             <axis xyz="0 1 0" />
-            <limit effort="270.0" velocity="2.09439510" lower="-2.617993878" upper="1.570796327" />
+            <limit effort="270.0" velocity="2.09439510" lower="-0.8" upper="0.8" />
         </joint>
         <joint name="torso_3" type="revolute">
@@ -642,5 +649,5 @@
             <origin rpy="0.0 0.0 0.0" xyz="0.0 0.0 0.0" />
             <axis xyz="1 0 0" />
-            <limit effort="120.0" velocity="3.141592654" lower="-0.523598776" upper="0.523598776" />
+            <limit effort="120.0" velocity="3.141592654" lower="-0.4" upper="0.4" />
         </joint>
         <joint name="torso_5" type="revolute">

File: urdf_rby/urdf/robots/rby_gazebo.urdf.xacro (robot description, xacro)
@@ -2,5 +2,5 @@
 <robot xmlns:xacro="http://www.ros.org/wiki/xacro" name="rby">
     <xacro:include filename="$(find urdf_rby)/urdf/robots/rby.urdf.xacro" />
-    <xacro:include filename="$(find gazebo_rby)/urdf/sensors/lidar_gazebo.urdf.xacro" />
+    <xacro:include filename="$(find urdf_rby)/urdf/sensors/lidar_gazebo.urdf.xacro" />
     <!-- Instantiate the robot -->
     <xacro:rby name="rby" use_sensors="true" />
